File: pcb/epd_board.brd (EAGLE design)
At the start: 35 x 21 mm, 83 parts, among them J1 SMT_JUMPER_2_NC_PASTE, J2 SMT_JUMPER_2_NC_PASTE, J3 SMT_JUMPER_2_NC_PASTE, P1 SMD-R1, P10 SMD-R1, P11 SMD-R1, P12 SMD-R1, P13 SMD-R1, P14 SMD-R1, P15 SMD-R1, P16 SMD-R1, P17 SMD-R1, P2 SMD-R1, P3 SMD-R1, P4 SMD-R1, P5 SMD-R1, P6 SMD-R1, P7 SMD-R1, P8 SMD-R1, P9 SMD-R1, Q1 NTNUS3171PZ, U1 WS4518D, U2 MIC5504, U3 ANT016008LCS2442MA2, U4 THD0515-30CL-SN, X1 XTAL_2016

Commit message: updated schematics and docs
Other:
- board text removed: "-+"
Changed lines of the file:
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@@
 <drawing>
 <settings>
-<setting alwaysvectorfont="yes"/>
+<setting alwaysvectorfont="no"/>
 <setting verticaltext="up"/>
 </settings>
@@
 </layers>
 <board>
-<fusionsync huburn="a.YnVzaW5lc3M6bXlpbWwxMA" projecturn="a.YnVzaW5lc3M6bXlpbWwxMCNEMjAyMTAzMDMzODg4NzY1MDY" f3durn="urn:adsk.wipprod:dm.lineage:7dAIbzZmRQqenzYGWIIWEQ" pcbguid="" lastpulledtime="" lastsyncedchangeguid="02835733-5250-87fb-8543-8cbafb76b1c9" latestrevisionid="89544a8e-cd4f-4ed2-9873-597686c39077" lastsyncedrevisionid="89544a8e-cd4f-4ed2-9873-597686c39077" lastboardhashguid="d7321c07-5051-ba8b-2582-4ba85838ef0e" lastpushedtime="2021-11-17T13:25:12Z" linktopcb3d="true"/>
+<fusionsync huburn="a.cGVyc29uYWw6dWUyY2VlYTJj" projecturn="a.cGVyc29uYWw6dWUyY2VlYTJjIzIwMTkwMTA1MTY4NTE3NjA2" f3durn="urn:adsk.wipprod:dm.lineage:teeD1Zy6ScGxuG0wg-2mqg" pcbguid="" lastpulledtime="" lastsyncedchangeguid="02835733-5250-87fb-8543-8cbafb76b1c9" latestrevisionid="584140a6-b60b-4cc1-8e0b-14660753efca" lastsyncedrevisionid="584140a6-b60b-4cc1-8e0b-14660753efca" lastboardhashguid="50f0dfe5-9fcb-5b63-dc8b-b158dc1b445e" lastpushedtime="2022-03-04T12:09:25Z" linktopcb3d="true"/>
 <plain>
 <wire x1="-14.5" y1="-10.5" x2="19.5" y2="-10.5" width="0" layer="20"/>
@@
 <wire x1="-15" y1="10" x2="-15" y2="-10" width="0" layer="20"/>
 <wire x1="-15" y1="-10" x2="-14.5" y2="-10.5" width="0" layer="20" curve="90"/>
-<text x="1.75" y="0" size="0.254" layer="21" font="vector" rot="R90" align="center">-+</text>
 <text x="6.8" y="0" size="0.8128" layer="134" font="vector" rot="MR270" align="center">Picoclick v3
 @maker.moekoe
@@
 <param name="layerSetup" value="(1*16)"/>
 <param name="mtCopper" value="0.035mm 0.0175mm 0.035mm 0.035mm 0.035mm 0.035mm 0.035mm 0.035mm 0.035mm 0.035mm 0.035mm 0.035mm 0.035mm 0.035mm 0.0175mm 0.035mm"/>
-<param name="mtIsolate" value="1.53mm 0.265mm 0.2mm 0.15mm 0.2mm 0.15mm 0.2mm 0.15mm 0.2mm 0.15mm 0.2mm 0.15mm 0.2mm 0.15mm 0.2mm"/>
+<param name="mtIsolate" value="0.93mm 0.265mm 0.2mm 0.15mm 0.2mm 0.15mm 0.2mm 0.15mm 0.2mm 0.15mm 0.2mm 0.15mm 0.2mm 0.15mm 0.2mm"/>
 <param name="mdWireWire" value="5mil"/>
 <param name="mdWirePad" value="4mil"/>
