File: pcb/epd_board.sch (EAGLE design)
At the start: 83 parts, among them J1 SMT_JUMPER_2_NC_PASTE, J2 SMT_JUMPER_2_NC_PASTE, J3 SMT_JUMPER_2_NC_PASTE, P1 SMD-R1, P10 SMD-R1, P11 SMD-R1, P12 SMD-R1, P13 SMD-R1, P14 SMD-R1, P15 SMD-R1, P16 SMD-R1, P17 SMD-R1, P2 SMD-R1, P3 SMD-R1, P4 SMD-R1, P5 SMD-R1, P6 SMD-R1, P7 SMD-R1, P8 SMD-R1, P9 SMD-R1, Q1 NTNUS3171PZ, U1 WS4518D, U2 MIC5504, U3 ANT016008LCS2442MA2, U4 THD0515-30CL-SN, X1 XTAL_2016

Commit message: updated schematics and docs
Other:
- note added: "250k"
Changed lines of the file:
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@@
 <wire x1="510.54" y1="106.68" x2="510.54" y2="60.96" width="0.508" layer="97" style="longdash"/>
 <text x="429.26" y="101.6" size="2.54" layer="97" font="vector" ratio="20">USER BUTTON</text>
+<text x="373.38" y="180.34" size="1.27" layer="98">250k</text>
 </plain>
 <instances>
