File: pcb/paperclick_v1.brd (EAGLE design)
At the start: 35 x 21 mm, 83 parts, among them J1 SMT_JUMPER_2_NC_PASTE, J2 SMT_JUMPER_2_NC_PASTE, J3 SMT_JUMPER_2_NC_PASTE, P1 SMD-R1, P10 SMD-R1, P11 SMD-R1, P12 SMD-R1, P13 SMD-R1, P14 SMD-R1, P15 SMD-R1, P16 SMD-R1, P17 SMD-R1, P2 SMD-R1, P3 SMD-R1, P4 SMD-R1, P5 SMD-R1, P6 SMD-R1, P7 SMD-R1, P8 SMD-R1, P9 SMD-R1, Q1 NTNUS3171PZ, U1 WS4518D, U2 MIC5504, U3 ANT016008LCS2442MA2, U4 THD0515-30CL-SN, X1 XTAL_2016

Commit message: updated schematics with correct values for the matching network
Parts:
- C22, C23: value tbd -> (none)
Changed lines of the file:
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@@
 <drawing>
 <settings>
-<setting alwaysvectorfont="no"/>
+<setting alwaysvectorfont="yes"/>
 <setting verticaltext="up"/>
 </settings>
@@
 </layers>
 <board>
-<fusionsync huburn="a.cGVyc29uYWw6dWUyY2VlYTJj" projecturn="a.cGVyc29uYWw6dWUyY2VlYTJjIzIwMTkwMTA1MTY4NTE3NjA2" f3durn="urn:adsk.wipprod:dm.lineage:teeD1Zy6ScGxuG0wg-2mqg" pcbguid="" lastpulledtime="" lastsyncedchangeguid="02835733-5250-87fb-8543-8cbafb76b1c9" latestrevisionid="584140a6-b60b-4cc1-8e0b-14660753efca" lastsyncedrevisionid="584140a6-b60b-4cc1-8e0b-14660753efca" lastboardhashguid="50f0dfe5-9fcb-5b63-dc8b-b158dc1b445e" lastpushedtime="2022-03-04T12:09:25Z" linktopcb3d="true"/>
+<fusionsync huburn="a.cGVyc29uYWw6dWUyY2VlYTJj" projecturn="a.cGVyc29uYWw6dWUyY2VlYTJjIzIwMTkwMTA1MTY4NTE3NjA2" f3durn="urn:adsk.wipprod:dm.lineage:teeD1Zy6ScGxuG0wg-2mqg" pcbguid="" lastpulledtime="" lastsyncedchangeguid="02835733-5250-87fb-8543-8cbafb76b1c9" latestrevisionid="584140a6-b60b-4cc1-8e0b-14660753efca" lastsyncedrevisionid="584140a6-b60b-4cc1-8e0b-14660753efca" lastboardhashguid="50f0dfe5-9fcb-5b63-dc8b-b158dc1b445e" lastpushedtime="2022-03-04T12:09:25Z" linktopcb3d="false"/>
 <plain>
 <wire x1="-14.5" y1="-10.5" x2="19.5" y2="-10.5" width="0" layer="20"/>
@@
 <element name="BAT+" library="iml_elc" package="SOLDERPAD_1.5X1.0" value="TP/SP-1.5X1.0" x="11.5" y="-8.5" smashed="yes" rot="R90"/>
 <element name="BAT-" library="iml_elc" package="SOLDERPAD_1.5X1.0" value="TP/SP-1.5X1.0" x="11.5" y="-6.5" smashed="yes" rot="R90"/>
-<element name="C23" library="moekoe_rcl" library_urn="urn:adsk.eagle:library:34187148" package="C0201" package3d_urn="urn:adsk.eagle:package:34200839/2" value="tbd" x="-11.8" y="9.4" smashed="yes" rot="R90">
+<element name="C23" library="moekoe_rcl" library_urn="urn:adsk.eagle:library:34187148" package="C0201" package3d_urn="urn:adsk.eagle:package:34200839/2" value="" x="-11.8" y="9.4" smashed="yes" rot="R90">
 <attribute name="NAME" x="-11.8" y="9.273" size="0.254" layer="25" font="vector" align="bottom-center"/>
 </element>
-<element name="C22" library="moekoe_rcl" library_urn="urn:adsk.eagle:library:34187148" package="C0201" package3d_urn="urn:adsk.eagle:package:34200839/2" value="tbd" x="-10.2" y="9.4" smashed="yes" rot="R90">
+<element name="C22" library="moekoe_rcl" library_urn="urn:adsk.eagle:library:34187148" package="C0201" package3d_urn="urn:adsk.eagle:package:34200839/2" value="" x="-10.2" y="9.4" smashed="yes" rot="R90">
 <attribute name="NAME" x="-10.2" y="9.273" size="0.254" layer="25" font="vector" align="bottom-center"/>
 </element>
